File: hardware/kicad/eeg-frontend/input_protection.kicad_sch (KiCad schematic)
At the start: 16 parts, among them CN3 1000pF, CN4 1000pF, CN5 1000pF, CN6 1000pF, CN7 1000pF, U10 TPD4E1B06DCKR, U11 TPD4E1B06DCKR, U2 TPD4E1B06DCKR, U7 TPD4E1B06DCKR, U8 TPD4E1B06DCKR, U9 TPD4E1B06DCKR

Commit message: Assign footprints to schematic components
Parts:
- CN3, CN4, CN5, CN6, CN7: footprint (none) -> myLibrary:C_Array_Convex_4x0612
- RN1, RN2, RN3, RN4, RN5: footprint (none) -> Resistor_SMD:R_Cat16-4
Changed lines of the file:
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@@
 			)
 		)
-		(property "Footprint" ""
+		(property "Footprint" "Resistor_SMD:R_Cat16-4"
 			(at 97.79 150.495 90)
 			(hide yes)
@@
 			)
 		)
-		(property "Footprint" ""
+		(property "Footprint" "myLibrary:C_Array_Convex_4x0612"
 			(at 118.872 100.33 90)
 			(hide yes)
@@
 			)
 		)
-		(property "Footprint" ""
+		(property "Footprint" "Resistor_SMD:R_Cat16-4"
 			(at 96.52 94.615 90)
 			(hide yes)
@@
 			)
 		)
-		(property "Footprint" ""
+		(property "Footprint" "Resistor_SMD:R_Cat16-4"
 			(at 95.25 40.005 90)
 			(hide yes)
@@
 			)
 		)
-		(property "Footprint" ""
+		(property "Footprint" "myLibrary:C_Array_Convex_4x0612"
 			(at 120.142 156.21 90)
 			(hide yes)
@@
 			)
 		)
-		(property "Footprint" ""
+		(property "Footprint" "myLibrary:C_Array_Convex_4x0612"
 			(at 261.112 105.41 90)
 			(hide yes)
@@
 			)
 		)
-		(property "Footprint" ""
+		(property "Footprint" "myLibrary:C_Array_Convex_4x0612"
 			(at 259.842 52.07 90)
 			(hide yes)
@@
 			)
 		)
-		(property "Footprint" ""
+		(property "Footprint" "myLibrary:C_Array_Convex_4x0612"
 			(at 117.602 45.72 90)
 			(hide yes)
@@
 			)
 		)
-		(property "Footprint" ""
+		(property "Footprint" "Resistor_SMD:R_Cat16-4"
 			(at 237.49 46.355 90)
 			(hide yes)
@@
 			)
 		)
-		(property "Footprint" ""
+		(property "Footprint" "Resistor_SMD:R_Cat16-4"
 			(at 238.76 99.695 90)
 			(hide yes)

Commit message: 一旦できたと思ったPCB。 しかしPMODのコネクタの位置が左右で逆で、このまま刺すとGNDの一に通常のデータ信号的なのが来てしまう。
Connections:
- net GND renamed AGND
Changed lines of the file:
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@@
 			)
 		)
-		(property "Value" "GND"
-			(at 251.46 95.25 0)
+		(property "Value" "AGND"
+			(at 254 97.79 0)
 			(show_name no)
 			(do_not_autoplace no)
@@
 					(size 0.762 0.762)
 				)
+				(justify right)
 			)
 		)
@@
 			)
 		)
-		(property "Value" "GND"
-			(at 109.22 116.84 0)
-			(show_name no)
-			(do_not_autoplace no)
-			(effects
-				(font
-					(size 1.27 1.27)
-				)
+		(property "Value" "AGND"
+			(at 111.76 113.0299 0)
+			(show_name no)
+			(do_not_autoplace no)
+			(effects
+				(font
+					(size 1.27 1.27)
+				)
+				(justify left)
 			)
 		)
@@
 			)
 		)
-		(property "Value" "GND"
-			(at 251.46 121.92 0)
-			(show_name no)
-			(do_not_autoplace no)
-			(effects
-				(font
-					(size 1.27 1.27)
-				)
+		(property "Value" "AGND"
+			(at 254 118.1099 0)
+			(show_name no)
+			(do_not_autoplace no)
+			(effects
+				(font
+					(size 1.27 1.27)
+				)
+				(justify left)
 			)
 		)
@@
 			)
 		)
-		(property "Value" "GND"
-			(at 110.49 172.72 0)
-			(show_name no)
-			(do_not_autoplace no)
-			(effects
-				(font
-					(size 1.27 1.27)
-				)
+		(property "Value" "AGND"
+			(at 113.03 168.9099 0)
+			(show_name no)
+			(do_not_autoplace no)
+			(effects
+				(font
+					(size 1.27 1.27)
+				)
+				(justify left)
 			)
 		)
@@
 		(in_pos_files yes)
 		(dnp no)
-		(fields_autoplaced yes)
 		(property "Reference" "#PWR010"
 			(at 107.95 63.5 0)
@@
 			)
 		)
-		(property "Value" "GND"
-			(at 107.95 62.23 0)
-			(show_name no)
-			(do_not_autoplace no)
-			(effects
-				(font
-					(size 1.27 1.27)
-				)
+		(property "Value" "AGND"
+			(at 106.172 60.706 0)
+			(show_name no)
+			(do_not_autoplace no)
+			(effects
+				(font
+					(size 1.27 1.27)
+				)
+				(justify left)
 			)
 		)
@@
 			)
 		)
-		(property "Value" "GND"
-			(at 185.42 143.51 0)
+		(property "Value" "AGND"
+			(at 189.23 139.7 90)
 			(show_name no)
 			(do_not_autoplace no)
@@
 			)
 		)
-		(property "Value" "GND"
-			(at 250.19 68.58 0)
-			(show_name no)
-			(do_not_autoplace no)
-			(effects
-				(font
-					(size 1.27 1.27)
-				)
+		(property "Value" "AGND"
+			(at 252.73 64.7699 0)
+			(show_name no)
+			(do_not_autoplace no)
+			(effects
+				(font
+					(size 1.27 1.27)
+				)
+				(justify left)
 			)
 		)
@@
 			)
 		)
-		(property "Value" "GND"
-			(at 185.42 138.43 0)
+		(property "Value" "AGND"
+			(at 189.23 134.62 90)
 			(show_name no)
 			(do_not_autoplace no)
@@
 			)
 		)
-		(property "Value" "GND"
+		(property "Value" "AGND"
 			(at 248.412 90.17 0)
 			(show_name no)
@@
 			)
 		)
-		(property "Value" "GND"
+		(property "Value" "AGND"
 			(at 229.108 90.17 0)
 			(show_name no)
